Commit message: Update final.xacro

File: extract_project/final_description/urdf/final.xacro (robot description, xacro)
@@ -108,5 +108,5 @@
   <parent link="base_link"/>
   <child link="right__1__1"/>
-  <axis xyz="-0.0 1.0 0.0"/>
+  <axis xyz="0.0 1.0 0.0"/>
 </joint>
 <joint name="Rev2" type="continuous">
@@ -114,5 +114,5 @@
   <parent link="base_link"/>
   <child link="left__2__1"/>
-  <axis xyz="-0.0 1.0 0.0"/>
+  <axis xyz="0.0 1.0 0.0"/>
 </joint>
 <joint name="Rev3" type="continuous">
@@ -120,5 +120,5 @@
   <parent link="mount__3__1"/>
   <child link="lidar__4__1"/>
-  <axis xyz="-0.0 0.0 1.0"/>
+  <axis xyz="0.0 0.0 1.0"/>
 </joint>
 <joint name="Rigid4" type="fixed">
